File: pcb/pcb.kicad_sch (KiCad schematic)
At the start: 113 parts, among them J1 MJ-4PP-9, J2 MJ-4PP-9, J3 USB_C_Receptacle_USB2.0_16P, J4 USB to TTL, J5 Conn_01x03, J6 Conn_01x03, SW1 KEY_SW, SW10 KEY_SW, SW11 KEY_SW, SW12 KEY_SW, SW13 KEY_SW, SW14 KEY_SW, SW15 KEY_SW, SW16 KEY_SW, SW17 KEY_SW, SW18 KEY_SW, SW19 KEY_SW, SW2 KEY_SW, SW20 KEY_SW, SW21 KEY_SW, SW22 KEY_SW, SW23 KEY_SW, SW24 KEY_SW, SW25 KEY_SW, SW26 KEY_SW, SW27 RotaryEncoder, SW3 KEY_SW, SW30 KEY_SW, SW31 KEY_SW, SW32 KEY_SW, SW33 KEY_SW, SW34 KEY_SW, SW35 KEY_SW, SW36 KEY_SW, SW37 KEY_SW, SW38 KEY_SW, SW39 KEY_SW, SW4 KEY_SW, SW40 KEY_SW, SW41 KEY_SW, SW42 KEY_SW, SW43 KEY_SW, SW44 KEY_SW, SW45 KEY_SW, SW46 KEY_SW, SW47 KEY_SW, SW48 KEY_SW, SW49 KEY_SW, SW5 KEY_SW, SW50 KEY_SW, SW51 KEY_SW, SW52 KEY_SW, SW53 KEY_SW, SW54 KEY_SW, SW6 KEY_SW, SW60 RESET_SW, SW61 BOOT_SW, SW7 KEY_SW, SW8 KEY_SW, SW9 KEY_SW, SW６２1 DIP_SW, U1 ESP32-S3-WROOM-1, U2 TPS1117LV33S, U3 USBLC6-2SC6

Commit message: put M2 hole
Parts:
- BT1: footprint Connector_JST:JST_XH_S2B-XH-A_1x02_P2.50mm_Horizontal -> lib:JST_XH_S2B-XH-A_1x02_P2.50mm_Horizontal
- J4: footprint Connector_PinSocket_2.54mm:PinSocket_1x06_P2.54mm_Horizontal -> lib:PinSocket_1x06_P2.54mm_Horizontal
Changed lines of the file:
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@@
 			)
 		)
-		(property "Footprint" "Connector_PinSocket_2.54mm:PinSocket_1x06_P2.54mm_Horizontal"
+		(property "Footprint" "lib:PinSocket_1x06_P2.54mm_Horizontal"
 			(at 182.88 259.08 0)
 			(effects
@@
 			)
 		)
-		(property "Footprint" "Connector_JST:JST_XH_S2B-XH-A_1x02_P2.50mm_Horizontal"
+		(property "Footprint" "lib:JST_XH_S2B-XH-A_1x02_P2.50mm_Horizontal"
 			(at 254 198.501 90)
 			(effects

Commit message: completed ERC
Parts:
- D1, D10, D11, D12, D13, D14, D15, D16, D17, D18, D19, D2, D20, D21, D22, D23, D24, D25, D26, D27, D28, D29, D3, D4, D5, D6, D7, D8, D9: footprint keebio:Diode-dual -> lib:Diode-dual
- J1, J2: symbol kbd:MJ-4PP-9 -> lib:MJ-4PP-9
Connections:
- net rotaryA: now also U1.4 (IO4)
- net rotaryB: now also U1.5 (IO5)
- no-connect marks 15 -> 13
Other:
- moved on the sheet: BT1, C1, C2, C3, C4, C5, C6, C7, D28, D29, J1, J2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
